Commit message: add model robot in rviz

File: ros_workspace/src/robot_control/urdf/mobile_base.urdf.xacro (robot description, xacro)
@@ -13,10 +13,10 @@
   <link name="base_link">
     <inertial>
-      <origin xyz="-0.1 0 -0.1" rpy="0 0 0"/>
+      <origin xyz="0 0 0.275" rpy="0 0 0"/>
       <mass value="10.0"/>
       <inertia ixx="0.25" ixy="0.0" ixz="0.0" iyy="0.5" iyz="0.0" izz="0.05"/>
     </inertial>
     <visual>
-      <origin xyz="0 0 0" rpy="0 0 0"/>
+      <origin xyz="0 0 0.275" rpy="0 0 0"/>
       <geometry>
         <box size="0.5 0.5 0.3"/>
@@ -25,5 +25,5 @@
     </visual>
     <collision>
-      <origin xyz="0 0 0" rpy="0 0 0"/>
+      <origin xyz="0 0 0.275" rpy="0 0 0"/>
       <geometry>
         <box size="0.5 0.5 0.3"/>
@@ -34,7 +34,7 @@
   <link name="laser_link">
     <visual>
-      <origin xyz="0.01 0 0.2" rpy="0 0 0"/>
+      <origin xyz="0.01 0 0.0" rpy="0 0 0"/>
       <geometry>
-        <cylinder length="0.05" radius="0.03"/>
+        <cylinder length="0.05" radius="0.06"/>
       </geometry>
       <material name="red"/>
@@ -45,10 +45,10 @@
     <parent link="base_link"/>
     <child link="laser_link"/>
-    <origin xyz="0.01 0 0.2" rpy="0 0 0"/>
+    <origin xyz="0.01 0 0.475" rpy="0 0 0"/>
   </joint>
   <!-- Left Wheel -->
   <link name="left_wheel">
   <visual>
-    <origin xyz="0 0 0" rpy="0 0 0"/>
+    <origin xyz="0 0 0" rpy="1.5708 0 0"/>
     <geometry>
       <cylinder radius="0.125" length="0.05"/>
@@ -57,5 +57,5 @@
   </visual>
   <collision>
-    <origin xyz="0 0 0" rpy="0 0 0"/>
+    <origin xyz="0 0 0" rpy="1.5708 0 0"/>
     <geometry>
       <cylinder radius="0.125" length="0.05"/>
@@ -66,5 +66,5 @@
     <parent link="base_link"/>
     <child link="left_wheel"/>
-    <origin xyz="0.2 0.29 0.125" rpy="0 1.5707 1.5707"/>
+    <origin xyz="0.2 0.29 0.125" rpy="0 0 0"/>
     <axis xyz="0 1 0"/>
   </joint>
@@ -72,5 +72,5 @@
     <link name="right_wheel">
         <visual>
-            <origin xyz="0 0 0" rpy="0 0 0"/>
+            <origin xyz="0 0 0" rpy="1.5708 0 0"/>
             <geometry>
                 <cylinder radius="0.125" length="0.05"/>
@@ -79,5 +79,5 @@
         </visual>
         <collision>
-            <origin xyz="0 0 0" rpy="0 0 0"/>
+            <origin xyz="0 0 0" rpy="1.5708 0 0"/>
             <geometry>
                 <cylinder radius="0.125" length="0.05"/>
@@ -88,5 +88,5 @@
     <parent link="base_link"/>
     <child link="right_wheel"/>
-    <origin xyz="0.2 -0.29 0.125" rpy="0 1.5707 1.5707"/>
+    <origin xyz="0.2 -0.29 0.125" rpy="0 0 0"/>
     <axis xyz="0 1 0"/>
   </joint>
@@ -110,5 +110,5 @@
     <parent link="base_link"/>
     <child link="caster_wheel"/>
-    <origin xyz="-0.2 0 -0.125" rpy="0 0 0"/>
+    <origin xyz="-0.2 0 0.125" rpy="0 0 0"/>
     </joint>
 </robot>
